File: Oven Controller/Oven Controller.sch (KiCad schematic (older format))
At the start: 108 parts, among them IC1 ATMEGA328P-P, IC2 ATTINY85-P, J1 RJ12, P1 12V Pwr, P10 SCK, P11 MOSI, P12 MISO, P14 ICSP_POWER, P15 85_SCK, P16 85_MISO, P17 85_MOSI, P18 85_RESET, P2 9V Pwr, P3 WATCHDOG_RELAY, P4 OVEN_RELAY, P5 FAN, P6 THERMO, P7 SERIAL, P8 328P_RESET, P9 EXPAND, Q1 MPS2222A, Q2 MPS2222A, Q3 MPS2222A, Q4 MPS2222A, Q5 MPS2222A, Q6 MPS2222A, Q7 MPS2222A, Q8 MPS2222A, Q9 MPS2222A, U1 LD1117V33, U2 LM7805CT, U3 Logic_Level_Shift, U4 MAX31855KASA, Y1 16 MHz

Commit message: Initial PCB design with throughhole components. Layout not finilized.
Parts:
- added C?: 1nF, Personal:C_Disc_D5_P7, symbol C
Connections:
- net +5V: now also C?.1
- net GND: now also C?.2
Changed lines of the file:
@@
 	10700 1050 10700 1000
 Connection ~ 10700 1000
+$Comp
+L C C?
+U 1 1 57E8C8AB
+P 9600 1350
+F 0 "C?" H 9625 1450 50  0000 L CNN
+F 1 "1nF" H 9625 1250 50  0000 L CNN
+F 2 "Personal:C_Disc_D5_P7" H 9638 1200 50  0001 C CNN
+F 3 "" H 9600 1350 50  0000 C CNN
+	1    9600 1350
+	1    0    0    -1
+$EndComp
 $EndSCHEMATC
