File: Weather_Balloon/Board/Heater.sch (KiCad schematic (older format))
At the start: 38 parts, among them P12 Custom_HEAT, P13 SHT31_HEAT, P14 GPS_HEAT, P15 UV_HEAT, P16 TSL2561_HEAT, Q1 PSMN9R1-30YL,115, Q2 PSMN9R1-30YL,115, Q3 PSMN9R1-30YL,115, Q4 PSMN9R1-30YL,115, Q5 PSMN9R1-30YL,115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

Commit message: Updated PCB board for larger traces and more compact design.
Parts:
- R73, R74, R75: footprint Resistors_SMD:R_1206_HandSoldering -> Personal:R_1206_WIDE
Changed lines of the file:
@@
 F 0 "R73" V 1850 900 50  0000 L CNN
 F 1 "16" V 1950 950 50  0000 L CNN
-F 2 "Resistors_SMD:R_1206_HandSoldering" V 1880 1000 50  0001 C CNN
+F 2 "Personal:R_1206_WIDE" V 1880 1000 50  0001 C CNN
 F 3 "" H 1950 1000 50  0000 C CNN
 	1    1950 1000
@@
 F 0 "R74" V 2050 900 50  0000 L CNN
 F 1 "16" V 2150 950 50  0000 L CNN
-F 2 "Resistors_SMD:R_1206_HandSoldering" V 2080 1000 50  0001 C CNN
+F 2 "Personal:R_1206_WIDE" V 2080 1000 50  0001 C CNN
 F 3 "" H 2150 1000 50  0000 C CNN
 	1    2150 1000
@@
 F 0 "R75" V 2250 900 50  0000 L CNN
 F 1 "16" V 2350 950 50  0000 L CNN
-F 2 "Resistors_SMD:R_1206_HandSoldering" V 2280 1000 50  0001 C CNN
+F 2 "Personal:R_1206_WIDE" V 2280 1000 50  0001 C CNN
 F 3 "" H 2350 1000 50  0000 C CNN
 	1    2350 1000
