File: Weather_Balloon/Board/Aux.sch (KiCad schematic (older format))
At the start: 78 parts, among them P11 UV_ADC, P17 LSM9DS1, P18 PIEZO, P19 MICRO_SD_CARD, P20 LANDING_LED, P21 DS18B20, P23 EXT_SENSORS, P26 MS5607, P27 GPS, P28 5V_BOOST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

Commit message: Updated PCB board for larger traces and more compact design.
Parts:
- P23: footprint Pin_Headers:Pin_Header_Straight_1x05 -> Pin_Headers:Pin_Header_Straight_1x03; symbol CONN_01X05 -> CONN_01X03
- U5: footprint Personal:FUEL_GAUGE_BACK -> Personal:FUEL_GAUGE_ALL
Connections:
- net +3V3: now also C23.1
- net +5V: now also C22.1
- net SHT_31_PWR: now also P23.2 (P2); no longer P23.3 (P3)
- net at Q13.2 (D): now also P23.3 (P3); no longer P23.4 (P4)
Other:
- moved on the sheet: C22, C23
Changed lines of the file:
@@
 L +3.3V #PWR047
 U 1 1 57E87428
-P 7750 3000
-F 0 "#PWR047" H 7750 2850 50  0001 C CNN
-F 1 "+3.3V" V 7750 3250 50  0000 C CNN
-F 2 "" H 7750 3000 50  0000 C CNN
-F 3 "" H 7750 3000 50  0000 C CNN
-	1    7750 3000
+P 7450 3000
+F 0 "#PWR047" H 7450 2850 50  0001 C CNN
+F 1 "+3.3V" V 7450 3250 50  0000 C CNN
+F 2 "" H 7450 3000 50  0000 C CNN
+F 3 "" H 7450 3000 50  0000 C CNN
+	1    7450 3000
 	0    -1   -1   0
 $EndComp
@@
 DOF_POWER
 $Comp
-L CONN_01X05 P23
+L CONN_01X03 P23
 U 1 1 57EA9852
 P 10050 3450
 F 0 "P23" H 10128 3491 50  0000 L CNN
 F 1 "EXT_SENSORS" H 9850 3150 50  0000 L CNN
-F 2 "Pin_Headers:Pin_Header_Straight_1x05" H 10050 3450 50  0001 C CNN
+F 2 "Pin_Headers:Pin_Header_Straight_1x03" H 10050 3450 50  0001 C CNN
 F 3 "" H 10050 3450 50  0000 C CNN
 	1    10050 3450
@@
 L C_Small C22
 U 1 1 57EA9858
-P 9650 4000
-F 0 "C22" H 9700 4100 50  0000 L CNN
-F 1 "0.1uF" H 9700 3900 50  0000 L CNN
-F 2 "Capacitors_SMD:C_1206_HandSoldering" H 9650 4000 50  0001 C CNN
-F 3 "" H 9650 4000 50  0000 C CNN
-	1    9650 4000
+P 7550 3550
+F 0 "C22" H 7600 3650 50  0000 L CNN
+F 1 "0.1uF" H 7600 3450 50  0000 L CNN
+F 2 "Capacitors_SMD:C_1206_HandSoldering" H 7550 3550 50  0001 C CNN
+F 3 "" H 7550 3550 50  0000 C CNN
+	1    7550 3550
 	-1   0    0    -1
 $EndComp
@@
 L +5V #PWR066
 U 1 1 57EA9BCA
-P 7750 3200
-F 0 "#PWR066" H 7750 3050 50  0001 C CNN
-F 1 "+5V" V 7765 3328 50  0000 L CNN
-F 2 "" H 7750 3200 50  0000 C CNN
-F 3 "" H 7750 3200 50  0000 C CNN
-	1    7750 3200
+P 7450 3200
+F 0 "#PWR066" H 7450 3050 50  0001 C CNN
+F 1 "+5V" V 7465 3328 50  0000 L CNN
+F 2 "" H 7450 3200 50  0000 C CNN
+F 3 "" H 7450 3200 50  0000 C CNN
+	1    7450 3200
 	0    -1   -1   0
 $EndComp
-Text GLabel 7750 3300 0    50   Input ~ 0
+Text GLabel 7450 3300 0    50   Input ~ 0
 SCL_5
-Text GLabel 7750 3100 0    50   BiDi ~ 0
+Text GLabel 7450 3100 0    50   BiDi ~ 0
 SDA_5
 $Comp
@@
 F 0 "U5" H 2450 6550 50  0000 C CNN
 F 1 "FUEL_GAUGE" H 2650 6150 50  0000 C CNN
-F 2 "Personal:FUEL_GAUGE_BACK" H 2675 6100 50  0001 C CNN
+F 2 "Personal:FUEL_GAUGE_ALL" H 2675 6100 50  0001 C CNN
 F 3 "" H 2675 6100 50  0001 C CNN
 	1    2650 6350
@@
 Text GLabel 1700 3700 0    50   Output ~ 0
 UV_PWR
-Text GLabel 9600 3250 0    50   Output ~ 0
+Text GLabel 9600 3350 0    50   Output ~ 0
 UV_PWR
 $Comp
 L C_Small C23
 U 1 1 57E9FD89
-P 9800 4000
-F 0 "C23" H 9850 4100 50  0000 L CNN
-F 1 "0.1uF" H 9850 3900 50  0000 L CNN
-F 2 "Capacitors_SMD:C_1206_HandSoldering" H 9800 4000 50  0001 C CNN
-F 3 "" H 9800 4000 50  0000 C CNN
-	1    9800 4000
+P 7750 3550
+F 0 "C23" H 7800 3650 50  0000 L CNN
+F 1 "0.1uF" H 7800 3450 50  0000 L CNN
+F 2 "Capacitors_SMD:C_1206_HandSoldering" H 7750 3550 50  0001 C CNN
+F 3 "" H 7750 3550 50  0000 C CNN
+	1    7750 3550
 	1    0    0    -1
 $EndComp
@@
 	9600 3350 9850 3350
 Wire Wire Line
-	9600 3250 9850 3250
-Wire Wire Line
-	7750 3300 7900 3300
-Wire Wire Line
-	7750 3100 7900 3100
+	7450 3300 7900 3300
+Wire Wire Line
+	7450 3100 7900 3100
 Wire Wire Line
 	1850 3700 1700 3700
@@
 Wire Wire Line
 	7900 1300 7900 2100
-Connection ~ 9650 4400
-Wire Wire Line
-	9800 4400 9800 4100
 Wire Wire Line
 	1850 3700 1850 3750
@@
 	4150 2550 4450 2550
 Wire Wire Line
-	3000 3200 4200 3200
+	4200 3200 3000 3200
 Wire Wire Line
 	6250 5250 6500 5250
@@
 Connection ~ 7500 950
 Wire Wire Line
-	7500 1000 7500 950
+	7500 950  7500 1000
 Connection ~ 7700 950
 Wire Wire Line
-	7700 1000 7700 950
+	7700 950  7700 1000
 Connection ~ 7050 950
 Wire Wire Line
@@
 Connection ~ 3000 3050
 Wire Wire Line
-	3050 3050 3000 3050
+	3000 3050 3050 3050
 Connection ~ 3000 2950
 Wire Wire Line
-	3050 2950 3000 2950
+	3000 2950 3050 2950
 Connection ~ 3000 2850
 Wire Wire Line
@@
 Connection ~ 4200 2850
 Wire Wire Line
-	4150 2850 4200 2850
+	4200 2850 4150 2850
 Connection ~ 4200 2950
 Wire Wire Line
-	4150 2950 4200 2950
+	4200 2950 4150 2950
 Connection ~ 4200 3050
 Wire Wire Line
-	4150 3050 4200 3050
+	4200 3050 4150 3050
 Connection ~ 4200 3200
 Wire Wire Line
-	3000 2750 3000 3200
-Wire Wire Line
-	3050 2750 3000 2750
+	3000 3200 3000 2750
+Wire Wire Line
+	3000 2750 3050 2750
 Wire Wire Line
 	4200 2650 4200 3300
@@
 Wire Wire Line
 	9850 3550 9300 3550
-Connection ~ 9650 3650
-Wire Wire Line
-	9650 3900 9650 3650
-Wire Wire Line
-	9600 3650 9850 3650
 Wire Wire Line
 	9300 3550 9300 3800
-Connection ~ 9300 4400
-Wire Wire Line
-	9650 4400 9650 4100
 Connection ~ 8950 4400
 Wire Wire Line
-	8950 4400 9800 4400
+	8950 4400 9300 4400
 Wire Wire Line
 	8550 4000 8600 4000
@@
 	8950 4350 8950 4450
 Wire Wire Line
-	9300 4200 9300 4400
+	9300 4400 9300 4200
 Connection ~ 4250 900
 Wire Wire Line
@@
 Connection ~ 1250 7000
 Wire Wire Line
-	1250 7050 1250 7000
+	1250 7000 1250 7050
 Wire Wire Line
 	1250 7400 1250 7350
@@
 Connection ~ 1250 6000
 Wire Wire Line
-	1250 6050 1250 6000
+	1250 6000 1250 6050
 Wire Wire Line
 	1250 6400 1250 6350
@@
 Connection ~ 1250 5000
 Wire Wire Line
-	1250 5050 1250 5000
+	1250 5000 1250 5050
 Wire Wire Line
 	1250 5400 1250 5350
@@
 	9600 3450 9850 3450
 Wire Wire Line
-	9800 3900 9800 3350
-Connection ~ 9800 3350
-Wire Wire Line
-	7750 3200 7900 3200
-Wire Wire Line
-	7900 3000 7750 3000
+	7450 3200 7900 3200
+Wire Wire Line
+	7900 3000 7450 3000
 $Comp
 L CONN_01X01 P11
@@
 Wire Wire Line
 	7750 2550 7900 2550
+$Comp
+L GND #PWR087
+U 1 1 57F0A628
+P 7550 3750
+F 0 "#PWR087" H 7550 3500 50  0001 C CNN
+F 1 "GND" H 7555 3577 50  0000 C CNN
+F 2 "" H 7550 3750 50  0000 C CNN
+F 3 "" H 7550 3750 50  0000 C CNN
+	1    7550 3750
+	1    0    0    -1
+$EndComp
+Wire Wire Line
+	7750 3650 7750 3700
+Wire Wire Line
+	7750 3700 7550 3700
+Wire Wire Line
+	7550 3650 7550 3750
+Connection ~ 7550 3700
+Wire Wire Line
+	7550 3450 7550 3200
+Connection ~ 7550 3200
+Wire Wire Line
+	7750 3450 7750 3000
+Connection ~ 7750 3000
 $EndSCHEMATC

Commit message: PID control and beginning of altitude alarm.
Other:
- note added: "DS18B20s draw parasitic power. \nAlso, MOSFET without capacitor \nacross DS18B20 will not communicate \nfor some reason."
Changed lines of the file:
@@
 	7750 3450 7750 3000
 Connection ~ 7750 3000
+Text Notes 4100 4100 0    50   ~ 0
+DS18B20s draw parasitic power. \nAlso, MOSFET without capacitor \nacross DS18B20 will not communicate \nfor some reason.
 $EndSCHEMATC

Commit message: After flight data retrieval
Other:
- note added: "DS18B20s draw parasitic power."
- note removed: "DS18B20s draw parasitic power. \nAlso, MOSFET without capacitor \nacross DS18B20 will not communicate \nfor some reason."
Changed lines of the file:
@@
 	7750 3450 7750 3000
 Connection ~ 7750 3000
-Text Notes 4100 4100 0    50   ~ 0
-DS18B20s draw parasitic power. \nAlso, MOSFET without capacitor \nacross DS18B20 will not communicate \nfor some reason.
+Text Notes 4350 3850 0    50   ~ 0
+DS18B20s draw parasitic power.
 $EndSCHEMATC
